File: design_files/AST1037.brd (EAGLE design)
At the start: 10 x 50 mm, 13 parts, among them J1 SM05B, U1 ATTINY25

Commit message: updated documentation
Parts:
- added R2: 10.0K, tinycircuits:0402
- C1: value 10uF -> 1uF
- R1: value 0.0 -> 1.00K
- R3: value 10.0K -> 10K
- moved R3 10.1 mm to (15.7, 18.2), turned to 270 degrees
- moved R1 3.00 mm to (18.3, 10.8)
- moved C1 3.00 mm to (10.8, 9.10)
- moved C2 3.00 mm to (13.3, 11.2)
- moved J1 3.00 mm to (15.0, 7.33)
- moved TP1 3.00 mm to (11.6, 14.3)
- moved TP2 3.00 mm to (11.6, 12.6)
- moved TP3 3.00 mm to (11.6, 10.9)
- moved TP5 3.00 mm to (11.6, 16.0)
- moved TP6 3.00 mm to (11.6, 7.50)
- moved U1 3.00 mm to (15.0, 14.3)
- moved TP4 3.00 mm to (11.6, 9.20)
Connections:
- new net TEMP: R3.2, U1.3
- net GND: now also R3.1
- net RESET: now also R2.1; no longer R3.1
- net VCC: now also R2.2; no longer R3.2
Routing:
- net TEMP: track 0.00 -> 4.09 mm
Other:
- board size 10 x 50 mm -> 10 x 52 mm
- board text added: "Wireling Soil Moisture"
- board text removed: "Soil Moisture Sensor"
- board text removed: "TinySaber R3"
