File: design_files/AST1037.sch (EAGLE design)
At the start: 12 parts, among them J1 SM05B, U1 ATTINY25

Commit message: updated documentation
Parts:
- added R2: 10.0K, tinycircuits:AS-ITM-00032
- C1: value 10uF -> 1uF; device tinycircuits:AS-ITM-00002 -> tinycircuits:AS-ITM-00410; PARTNO (none) -> AS-ITM-00410; VALUE (none) -> 1uF
- R1: value 0.0 -> 1.00K; device tinycircuits:AS-ITM-00076 -> tinycircuits:AS-ITM-00003; PARTNO (none) -> AS-ITM-00003; VALUE (none) -> 1.00K
- R3: value 10.0K -> 10K; device tinycircuits:AS-ITM-00032 -> tinycircuits:AS-ITM-00524
Connections:
- new net TEMP: R3.2, U1.PB4
- net GND: now also R3.1
- net RESET: now also R2.1; no longer R3.1
- net VCC: now also R2.2; no longer R3.2
Other:
- note added: "Variant: Standard - R"
- note added: "Wireling Soil Moisture"
- note removed: "Soil Moisture Sensor"
- note removed: "Variant: Standard"
Changed lines of the file:
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@@
 <layer number="59" name="Invisible" color="7" fill="1" visible="no" active="no"/>
 <layer number="61" name="stand" color="7" fill="1" visible="no" active="no"/>
+<layer number="88" name="SimResults" color="9" fill="1" visible="yes" active="yes"/>
+<layer number="89" name="SimProbes" color="9" fill="1" visible="yes" active="yes"/>
 <layer number="90" name="Modules" color="5" fill="1" visible="yes" active="yes"/>
 <layer number="91" name="Nets" color="2" fill="1" visible="yes" active="yes"/>
@@
 <layer number="158" name="bResistor" color="7" fill="1" visible="no" active="yes"/>
 <layer number="159" name="henwayCAP" color="13" fill="1" visible="yes" active="yes"/>
+<layer number="160" name="IDFDebug" color="7" fill="1" visible="yes" active="yes"/>
 <layer number="191" name="mNets" color="7" fill="1" visible="yes" active="yes"/>
 <layer number="192" name="mBusses" color="7" fill="1" visible="yes" active="yes"/>
@@
 <part name="GND1" library="tinycircuits" deviceset="GND" device=""/>
 <part name="P+1" library="tinycircuits" deviceset="VCC" device=""/>
-<part name="C1" library="tinycircuits" deviceset="AS-ITM-00002" device="" value="10uF"/>
+<part name="C1" library="tinycircuits" deviceset="AS-ITM-00410" device="" value="1uF">
+<attribute name="PARTNO" value="AS-ITM-00410"/>
+<attribute name="VALUE" value="1uF"/>
+</part>
 <part name="J1" library="tinycircuits" deviceset="AS-ITM-00340" device="" value="SM05B"/>
 <part name="P+2" library="tinycircuits" deviceset="VCC" device=""/>
 <part name="GND2" library="tinycircuits" deviceset="GND" device=""/>
-<part name="R1" library="tinycircuits" deviceset="AS-ITM-00076" device="" value="0.0"/>
+<part name="R1" library="tinycircuits" deviceset="AS-ITM-00003" device="" value="1.00K">
+<attribute name="PARTNO" value="AS-ITM-00003"/>
+<attribute name="VALUE" value="1.00K"/>
+</part>
 <part name="U1" library="tinycircuits" deviceset="AS-ITM-00330" device="" value="ATTINY25"/>
-<part name="R3" library="tinycircuits" deviceset="AS-ITM-00032" device="" value="10.0K"/>
+<part name="R2" library="tinycircuits" deviceset="AS-ITM-00032" device="" value="10.0K"/>
 <part name="P+4" library="tinycircuits" deviceset="VCC" device=""/>
 <part name="TP1" library="tinycircuits" deviceset="TEST_POINT" device=""/>
@@
 <part name="TP5" library="tinycircuits" deviceset="TEST_POINT" device=""/>
 <part name="TP6" library="tinycircuits" deviceset="TEST_POINT" device=""/>
+<part name="R3" library="tinycircuits" deviceset="AS-ITM-00524" device="" value="10K"/>
+<part name="GND3" library="tinycircuits" deviceset="GND" device=""/>
 </parts>
 <sheets>
 <sheet>
 <plain>
-<text x="340.868" y="17.272" size="3.556" layer="94" font="vector">Soil Moisture Sensor</text>
+<text x="340.868" y="17.272" size="3.556" layer="94" font="vector">Wireling Soil Moisture</text>
 <text x="327.152" y="6.35" size="3.556" layer="94" font="vector">AS-SCH-AST1037</text>
 <text x="416.56" y="6.858" size="3.556" layer="94" font="vector">1</text>
@@
 <text x="68.58" y="73.66" size="1.778" layer="96">Hand Populated: -</text>
 <text x="68.58" y="71.12" size="1.778" layer="96">Hand Soldered: -</text>
-<text x="68.58" y="78.74" size="1.778" layer="96">Variant: Standard</text>
+<text x="68.58" y="78.74" size="1.778" layer="96">Variant: Standard - R</text>
 <text x="68.58" y="68.58" size="1.778" layer="96">Notes: -</text>
 </plain>
@@
 <instance part="R1" gate="G$1" x="223.52" y="137.16" rot="R180"/>
 <instance part="U1" gate="G$1" x="177.8" y="157.48"/>
-<instance part="R3" gate="G$1" x="205.74" y="149.86"/>
+<instance part="R2" gate="G$1" x="205.74" y="149.86"/>
 <instance part="P+4" gate="VCC" x="213.36" y="154.94" smashed="yes">
 <attribute name="VALUE" x="215.9" y="157.48" size="1.778" layer="96" rot="R180"/>
@@
 <attribute name="NAME" x="302.006" y="150.368" size="1.778" layer="96" rot="R180"/>
 </instance>
+<instance part="R3" gate="G$1" x="193.04" y="132.08" rot="R90"/>
+<instance part="GND3" gate="1" x="193.04" y="121.92"/>
 </instances>
 <busses>
@@
 <pinref part="TP6" gate="G$1" pin="1"/>
 </segment>
+<segment>
+<pinref part="R3" gate="G$1" pin="1"/>
+<wire x1="193.04" y1="127" x2="193.04" y2="124.46" width="0.1524" layer="91"/>
+<pinref part="GND3" gate="1" pin="GND"/>
+</segment>
 </net>
 <net name="VCC" class="0">
@@
 </segment>
 <segment>
-<pinref part="R3" gate="G$1" pin="2"/>
+<pinref part="R2" gate="G$1" pin="2"/>
 <pinref part="P+4" gate="VCC" pin="VCC"/>
 <wire x1="210.82" y1="149.86" x2="213.36" y2="149.86" width="0.1524" layer="91"/>
@@
 <wire x1="190.5" y1="149.86" x2="200.66" y2="149.86" width="0.1524" layer="91"/>
 <label x="193.04" y="149.86" size="1.778" layer="95"/>
-<pinref part="R3" gate="G$1" pin="1"/>
+<pinref part="R2" gate="G$1" pin="1"/>
 </segment>
 <segment>
@@
 </segment>
 </net>
+<net name="TEMP" class="0">
+<segment>
+<label x="193.04" y="139.7" size="1.778" layer="95"/>
+<wire x1="193.04" y1="137.16" x2="193.04" y2="139.7" width="0.1524" layer="91"/>
+<pinref part="R3" gate="G$1" pin="2"/>
+</segment>
+<segment>
+<pinref part="U1" gate="G$1" pin="PB4"/>
+<wire x1="190.5" y1="152.4" x2="200.66" y2="152.4" width="0.1524" layer="91"/>
+<label x="193.04" y="152.4" size="1.778" layer="95"/>
+</segment>
+</net>
